Commit message: tryna to push

File: catkin_ws/src/my_robot/urdf/my_robot.xacro (robot description, xacro)
@@ -118,5 +118,5 @@
 		<dynamics damping="1.0" friction="1.0"/>
 	</joint>
-	<link name='camera'>
+	<link name='camera_link'>
 		<visual>
 			<origin xyz="0 0 0" rpy="0 0 0"/>
@@ -143,8 +143,15 @@
 	<joint type='fixed' name='camera_joint'>
 		<origin xyz="0.2 0 0" rpy="0 0 0"/>
-		<child link="camera"/>
-		<parent link="chassis"/>
-		<axis xyz="0 1 0" rpy="0 0 0"/>
-	</joint>
+		<child link="camera_link"/>
+		<parent link="chassis"/>
+		<axis xyz="0 1 0" rpy="0 0 0"/>
+	</joint>
+	<joint name="camera_optical_joint" type="fixed">
+		<origin xyz="0 0 0" rpy="-1.5707 0 -1.5707"/>
+		<parent link="camera_link"/>
+		<child link="camera_link_optical"/>
+  	</joint>
+  	<link name="camera_link_optical">
+  	</link>
 	<link name='hokuyo'>
 		<visual>
@@ -176,4 +183,48 @@
 		<axis xyz="0 1 0" rpy="0 0 0"/>
 	</joint>
+	<!-- RGBD Camera -->
+  	<!--<gazebo reference="camera_link">
+		<sensor type="depth" name="camera1">
+		    <always_on>1</always_on>
+		    <update_rate>20.0</update_rate>
+		    <visualize>true</visualize>
+		    <camera>
+		        <horizontal_fov>1.047</horizontal_fov>
+		        <image>
+		            <width>640</width>
+		            <height>480</height>
+		            <format>R8G8B8</format>
+		        </image>
+		        <depth_camera>
+		        </depth_camera>
+		        <clip>
+		            <near>0.1</near>
+		            <far>20</far>
+		        </clip>
+		    </camera>
+		     <plugin name="camera_controller" filename="libgazebo_ros_openni_kinect.so">
+		        <alwaysOn>true</alwaysOn>
+		        <updateRate>10.0</updateRate>
+		        <cameraName>camera</cameraName>
+		        <frameName>camera_link_optical</frameName>
+		        <imageTopicName>rgb/image_raw</imageTopicName>
+		        <depthImageTopicName>depth/image_raw</depthImageTopicName>
+		        <pointCloudTopicName>depth/points</pointCloudTopicName>
+		        <cameraInfoTopicName>rgb/camera_info</cameraInfoTopicName>
+		        <depthImageCameraInfoTopicName>depth/camera_info</depthImageCameraInfoTopicName>
+		        <pointCloudCutoff>0.4</pointCloudCutoff>
+		            <hackBaseline>0.07</hackBaseline>
+		            <distortionK1>0.0</distortionK1>
+		            <distortionK2>0.0</distortionK2>
+		            <distortionK3>0.0</distortionK3>
+		            <distortionT1>0.0</distortionT1>
+		            <distortionT2>0.0</distortionT2>
+		        <CxPrime>0.0</CxPrime>
+		        <Cx>0.0</Cx>
+		        <Cy>0.0</Cy>
+		        <focalLength>0.0</focalLength>
+		        </plugin>
+		</sensor>
+  	</gazebo>-->
 	<gazebo reference="left_wheel">
 		<material>Gazebo/Green</material>
